Commit message: Added welding gun to robot description

File: weld_flow_description/urdf/mech/welding_gun_lorch_scancontrol_3000.urdf.xacro (robot description, xacro)
@@ -24,4 +24,15 @@
       </collision>
     </link>
+    <link name="tcp_welding_gun_link"/>
+    <joint name="tcp_welding_gun_joint" type="fixed">
+      <origin xyz="0.00132 -0.00363 0.42954" rpy="3.1416 -2.3561 -1.571"/>
+      <parent link="wrist_3_link"/>
+      <child link="tcp_welding_gun_link"/>
+    </joint>
+    <joint name="welding_gun_joint" type="fixed">
+      <origin xyz="0.0 0.0 0.0" rpy="0.0 0.0 0.0"/>
+      <parent link="tcp_welding_gun_link"/>
+      <child link="welding_gun_link"/>
+    </joint>
   </xacro:macro>
 </robot>

File: weld_flow_description/urdf/robots/ur10e.urdf.xacro (robot description, xacro)
@@ -33,3 +33,5 @@
         <origin xyz="0 0 0" rpy="0 0 0" />          <!-- position robot in the world -->
     </xacro:ur_robot>
+    <!--welding gun-->
+    <xacro:end_effector prefix="$(arg prefix)"/>
 </robot>
