Commit message: Configured Gazebo for ur10e

File: moveit_config/ur10e_moveit_config/config/ur10e.urdf.xacro (robot description, xacro)
@@ -2,8 +2,23 @@
 <robot xmlns:xacro="http://www.ros.org/wiki/xacro" name="ur10e">
     <xacro:arg name="initial_positions_file" default="initial_positions.yaml" />
+    <xacro:arg name="use_gazebo" default="false"/>
+    <xacro:arg name="use_mock_hardware" default="true"/>
     <!-- Import ur10e urdf file -->
     <xacro:include filename="$(find weld_flow_description)/urdf/robots/ur10e.urdf.xacro" />
-    <!-- Import control_xacro -->
-    <xacro:include filename="ur10e.ros2_control.xacro" />
-    <xacro:ur10e_ros2_control name="FakeSystem" initial_positions_file="$(arg initial_positions_file)"/>
+    <!-- Import generated control_xacro -->
+    <!--xacro:include filename="ur10e.ros2_control.xacro" /-->
+    <!--Import custom control xacro-->
+    <xacro:include filename="$(find weld_flow_description)/urdf/control/ur10_ros2_control.urdf.xacro"/>
+    <!--Import visual utils for gazebo arm-->
+    <xacro:include filename="$(find weld_flow_description)/urdf/gazebo/ur10e.urdf.xacro" />
+    <!--Import gazebo ros2_control plugin-->
+    <xacro:include filename="$(find weld_flow_description)/urdf/control/gazebo_sim.urdf.xacro"/>
+    <xacro:if value="$(arg use_gazebo)">
+        <xacro:ur10e_ros2_control initial_positions_file="$(arg initial_positions_file)" use_gazebo="$(arg use_gazebo)" use_mock_hardware="$(arg use_mock_hardware)"/>
+        <xacro:ur10_gazebo_utils/>
+        <xacro:load_gazebo_sim_ros2_control_plugin robot_name="ur10e"/>
+    </xacro:if>
+    <xacro:if value="$(arg use_mock_hardware)">
+        <xacro:ur10e_ros2_control initial_positions_file="$(arg initial_positions_file)" use_gazebo="$(arg use_gazebo)" use_mock_hardware="$(arg use_mock_hardware)"/>
+    </xacro:if>
 </robot>

File: weld_flow_description/urdf/mech/welding_gun_lorch_scancontrol_3000.urdf.xacro (robot description, xacro)
@@ -35,4 +35,13 @@
       <child link="welding_gun_link"/>
     </joint>
+    <gazebo reference="welding_gun_link">
+      <visual>
+        <material>
+          <ambient>0.5 0.5 0.5 1</ambient>
+          <diffuse>0.5 0.5 0.5 1</diffuse>
+          <specular>0.5 0.5 0.5 1</specular>
+        </material>
+      </visual>
+    </gazebo>
   </xacro:macro>
 </robot>

File: weld_flow_description/urdf/robots/ur10e.urdf.xacro (robot description, xacro)
@@ -1,8 +1,9 @@
 <?xml version="1.0"?>
 <robot xmlns:xacro="http://www.ros.org/wiki/xacro" name="ur10e">
+<!--Perhaps make this a macro...-->
     <xacro:arg name='prefix' default=""/>
     <xacro:arg name="ur_type" default="ur10e"/>
     <xacro:arg name="name" default="ur"/>
-    <xacro:arg name="force_abs_paths" default="false" />
+    <xacro:arg name="force_abs_paths" default="true" /> <!--When using gazebo set to true-->
     <xacro:arg name="joint_limit_params" default="$(find ur_description)/config/$(arg ur_type)/joint_limits.yaml"/>
     <xacro:arg name="kinematics_params" default="$(find ur_description)/config/$(arg ur_type)/default_kinematics.yaml"/>

Commit message: Configured top level xacro

File: moveit_config/ur10e_moveit_config/config/ur10e.urdf.xacro (robot description, xacro)
@@ -4,6 +4,46 @@
     <xacro:arg name="use_gazebo" default="false"/>
     <xacro:arg name="use_mock_hardware" default="true"/>
+    <xacro:arg name='prefix' default=""/>
+    <xacro:arg name="ur_type" default="ur10e"/>
+    <xacro:arg name="name" default="ur"/>
+    <xacro:arg name="force_abs_paths" default="false" /> <!--When using gazebo set to true-->
+    <xacro:arg name="joint_limit_params" default="$(find ur_description)/config/$(arg ur_type)/joint_limits.yaml"/>
+    <xacro:arg name="kinematics_params" default="$(find ur_description)/config/$(arg ur_type)/default_kinematics.yaml"/>
+    <xacro:arg name="physical_params" default="$(find ur_description)/config/$(arg ur_type)/physical_parameters.yaml"/>
+    <xacro:arg name="visual_params" default="$(find ur_description)/config/$(arg ur_type)/visual_parameters.yaml"/>
+    <xacro:arg name="transmission_hw_interface" default=""/>
+    <xacro:arg name="safety_limits" default="false"/>
+    <xacro:arg name="safety_pos_margin" default="0.15"/>
+    <xacro:arg name="safety_k_position" default="20"/>
+    <xacro:arg name="x" default="0"/>
+    <xacro:arg name="y" default="0"/>
+    <xacro:arg name="z" default="0"/>
+    <xacro:arg name="roll" default="0"/>
+    <xacro:arg name="pitch" default="0"/>
+    <xacro:arg name="yaw" default="0"/>
+    <xacro:include filename="$(find weld_flow_description)/urdf/mech/welding_gun_lorch_scancontrol_3000.urdf.xacro"/>
+    <xacro:include filename="$(find ur_description)/urdf/ur_macro.xacro"/>
+    <!-- create link fixed to the "world" -->
+    <link name="world" />
+    <!-- arm -->
+    <xacro:ur_robot
+        name="$(arg name)"
+        tf_prefix="$(arg prefix)"
+        parent="world"
+        joint_limits_parameters_file="$(arg joint_limit_params)"
+        kinematics_parameters_file="$(arg kinematics_params)"
+        physical_parameters_file="$(arg physical_params)"
+        visual_parameters_file="$(arg visual_params)"
+        safety_limits="$(arg safety_limits)"
+        safety_pos_margin="$(arg safety_pos_margin)"
+        safety_k_position="$(arg safety_k_position)"
+        force_abs_paths="$(arg force_abs_paths)"
+        >
+        <origin xyz="$(arg x) $(arg y) $(arg z)" rpy="$(arg roll) $(arg pitch) $(arg yaw)" />          <!-- position robot in the world -->
+    </xacro:ur_robot>
+    <!--welding gun-->
+    <xacro:end_effector prefix="$(arg prefix)"/>
     <!-- Import ur10e urdf file -->
-    <xacro:include filename="$(find weld_flow_description)/urdf/robots/ur10e.urdf.xacro" />
+    <!--xacro:include filename="$(find weld_flow_description)/urdf/robots/ur10e.urdf.xacro" /-->
     <!-- Import generated control_xacro -->
     <!--xacro:include filename="ur10e.ros2_control.xacro" /-->

Commit message: Added FT sensor for ur10e

File: moveit_config/ur10e_moveit_config/config/ur10e.urdf.xacro (robot description, xacro)
@@ -24,4 +24,6 @@
     <xacro:include filename="$(find weld_flow_description)/urdf/mech/welding_gun_lorch_scancontrol_3000.urdf.xacro"/>
     <xacro:include filename="$(find ur_description)/urdf/ur_macro.xacro"/>
+    <xacro:include filename="$(find weld_flow_description)/urdf/sensors/ft_sensor.urdf.xacro"/>
+    <xacro:include filename="$(find weld_flow_description)/urdf/control/ft_sensor_ros2_control.urdf.xacro"/>
     <!-- create link fixed to the "world" -->
     <link name="world" />
@@ -42,10 +44,8 @@
         <origin xyz="$(arg x) $(arg y) $(arg z)" rpy="$(arg roll) $(arg pitch) $(arg yaw)" />          <!-- position robot in the world -->
     </xacro:ur_robot>
+    <!--ft_sensor-->
+    <xacro:ft_sensor/>
     <!--welding gun-->
     <xacro:end_effector prefix="$(arg prefix)"/>
-    <!-- Import ur10e urdf file -->
-    <!--xacro:include filename="$(find weld_flow_description)/urdf/robots/ur10e.urdf.xacro" /-->
-    <!-- Import generated control_xacro -->
-    <!--xacro:include filename="ur10e.ros2_control.xacro" /-->
     <!--Import custom control xacro-->
     <xacro:include filename="$(find weld_flow_description)/urdf/control/ur10_ros2_control.urdf.xacro"/>

File: weld_flow_description/urdf/control/gazebo_sim.urdf.xacro (robot description, xacro)
@@ -4,5 +4,6 @@
             <gazebo>
             <plugin filename="gz_ros2_control-system" name="gz_ros2_control::GazeboSimROS2ControlPlugin">
-                <parameters>$(find ${robot_name}_moveit_config)/config/ros2_controllers.yaml</parameters>
+                <parameters>$(find ${robot_name}_moveit_config)/config/ros2_controllers.yaml</parameters> <!--Robot controllers-->
+                <parameters>$(find weld_flow_description)/config/sensors_controllers.yaml</parameters> <!--Sensor controllers-->
                 <ros>
                     <remapping>/controller_manager/robot_description:=/robot_description</remapping>

File: weld_flow_description/urdf/control/ur10_ros2_control.urdf.xacro (robot description, xacro)
@@ -51,4 +51,5 @@
                 </state_interface>
             </joint>
+            <xacro:ft_sensor_ros2_control/>
         </ros2_control>
     </xacro:macro>

File: weld_flow_description/urdf/mech/welding_gun_lorch_scancontrol_3000.urdf.xacro (robot description, xacro)
@@ -27,5 +27,5 @@
     <joint name="tcp_welding_gun_joint" type="fixed">
       <origin xyz="0.00132 -0.00363 0.42954" rpy="3.1416 -2.3561 -1.571"/>
-      <parent link="wrist_3_link"/>
+      <parent link="ft_sensor_link"/>
       <child link="tcp_welding_gun_link"/>
     </joint>

File: weld_flow_description/urdf/robots/ur10e.urdf.xacro (robot description, xacro)
@@ -16,4 +16,5 @@
     <xacro:include filename="$(find weld_flow_description)/urdf/mech/welding_gun_lorch_scancontrol_3000.urdf.xacro"/>
     <xacro:include filename="$(find ur_description)/urdf/ur_macro.xacro"/>
+    <xacro:include filename="$(find weld_flow_description)/urdf/sensors/ft_sensor.urdf.xacro"/>
     <!-- create link fixed to the "world" -->
     <link name="world" />
@@ -34,4 +35,6 @@
         <origin xyz="0 0 0" rpy="0 0 0" />          <!-- position robot in the world -->
     </xacro:ur_robot>
+    <!--ft_sensor-->
+    <xacro:ft_sensor/>
     <!--welding gun-->
     <xacro:end_effector prefix="$(arg prefix)"/>

Commit message: Parametrized ft_sensor

File: moveit_config/ur10e_moveit_config/config/ur10e.urdf.xacro (robot description, xacro)
@@ -45,5 +45,5 @@
     </xacro:ur_robot>
     <!--ft_sensor-->
-    <xacro:ft_sensor/>
+    <xacro:ft_sensor parent_link="tool0"/>
     <!--welding gun-->
     <xacro:end_effector prefix="$(arg prefix)"/>

File: weld_flow_description/urdf/robots/ur10e.urdf.xacro (robot description, xacro)
@@ -36,5 +36,5 @@
     </xacro:ur_robot>
     <!--ft_sensor-->
-    <xacro:ft_sensor/>
+    <xacro:ft_sensor parent_link="tool0"/>
     <!--welding gun-->
     <xacro:end_effector prefix="$(arg prefix)"/>

File: weld_flow_description/urdf/sensors/ft_sensor.urdf.xacro (robot description, xacro)
@@ -1,5 +1,5 @@
 <?xml version="1.0"?>
 <robot xmlns:xacro="http://www.ros.org/wiki/xacro">
-    <xacro:macro name="ft_sensor">
+    <xacro:macro name="ft_sensor" params="parent_link">
         <link name="ft_sensor_link">
             <inertial>
@@ -11,5 +11,5 @@
         <joint name="ft_sensor_joint" type="fixed">
             <origin xyz="0.0 0.0 0.0" rpy="0.0 0.0 0.0"/>
-            <parent link="tool0"/>
+            <parent link="${parent_link}"/> <!--tool0-->
             <child link="ft_sensor_link"/>
         </joint>
